File: assignments.kicad_sch (KiCad schematic)
At the start: 0 parts

Commit message: Update assignments.kicad_sch
Parts:
- added 8MHz: Y2, symbol Device:Crystal
- added C1, C10, C11, C3, C4: 10nF, symbol Device:C
- added C13, C14: 20pF, symbol Device:C
- added C2: 100nf, symbol Device:C
- added C20, c21: 10uF, symbol Device:C
- added D1, D2: LED, symbol Device:LED
- added P1: (no value), symbol Connector_Generic:Conn_02x03_Odd_Even
- added P2: SWD, symbol Connector:Conn_01x04_Pin
- added P3, P4: Header20, symbol Connector:Conn_01x20_Pin
- added R1, R5: 510R, symbol Device:R
- added R10: 4.7k, symbol Device:R
- added R11, R9: 20R, symbol Device:R
- added R2: 10k, symbol Device:R
- added R3, R4: 100k, symbol Device:R
- added R6: 1M, symbol Device:R
- added Rest: (no value), symbol Switch:SW_Push
- added U1: LM1117LD-3.3, Package_SON:WSON-8-1EP_4x4mm_P0.8mm_EP2.2x3mm, symbol Regulator_Linear:LM1117LD-3.3
- added U2: STM32F103C8T6, Package_QFP:LQFP-48_7x7mm_P0.5mm, symbol MCU_ST_STM32F1:STM32F103C8Tx
- added U3: USB_B_Micro, symbol Connector:USB_B_Micro
Connections:
- new net: R9.1, U3.3 (D+)
- new net: C1.1, P2.1 (Pin_1)
- new net: C1.2, P2.4 (Pin_4)
- new net: C2.1, R2.2, Rest.2
- new net: C2.2, Rest.1
- new net: P1.4 (Pin_4), R4.1
- new net: 8MHz.2, C13.1, R6.2
- new net: C13.2, C14.2
- new net: 8MHz.1, C14.1, R6.1
- new net: U2.23 (VSS), U2.35 (VSS), U2.47 (VSS), U2.8 (VSSA)
- new net: U2.24 (VDD), U2.36 (VDD), U2.48 (VDD), U2.9 (VDDA)
- new net: D2.1 (K), R5.1
- new net: R10.2, R11.2
- new net: D1.1 (K), R1.1
- new net: R11.1, U3.2 (D-)
- new net: U3.4 (ID), U3.5 (GND), U3.SH (Shield)
- new net: P1.3 (Pin_3), R3.2
- new net: P1.1 (Pin_1), P1.2 (Pin_2)
- new net +3.3V: R2.1, U1.5 (VO), U1.6 (VO), U1.7 (VO), U1.9 (VO), c21.1
- new net +5V: C20.1, R10.1, U1.2 (VI), U1.3 (VI), U1.4 (VI), U3.1 (VBUS)
- new net GND: C10.2, C11.2, C20.2, C3.2, C4.2, P1.5 (Pin_5), P1.6 (Pin_6), U1.1 (GND), c21.2
Other:
- note added: "105"
- note added: "10nF"
- note added: "5V --> 3.3V"
- note added: "5v"
- note added: "BOOT0"
- note added: "BOOT1"
- note added: "BOOTx"
- note added: "GND"
- note added: "J-Link OB"
- note added: "LED"
- note added: "MCU"
- note added: "NRST"
- note added: "OSCIN"
- note added: "OSCOUT"
- note added: "PA0"
- note added: "PA1"
- note added: "PA10"
- note added: "PA11"
- note added: "PA12"
- note added: "PA13"
- note added: "PA14"
- note added: "PA15"
- note added: "PA2"
- note added: "PA3"
- note added: "PA4"
- note added: "PA5"
- note added: "PA6"
- note added: "PA7"
- note added: "PA8"
- note added: "PA9"
- note added: "PB0"
- note added: "PB1"
- note added: "PB10"
- note added: "PB11"
- note added: "PB12"
- note added: "PB13"
- note added: "PB14"
- note added: "PB15"
- note added: "PB2/BOOT1"
- note added: "PB3"
- note added: "PB4"
- note added: "PB5"
- note added: "PB6"
- note added: "PB7"
- note added: "PB8"
- note added: "PB9"
- note added: "PC13"
- note added: "PC14"
- note added: "PC15"
- note added: "RES"
- note added: "RESET"
- note added: "SWDCLK"
- note added: "SWDIO"
- note added: "USB"
- note added: "VBAT"
- note added: "VCC3V3"
- company: (none) -> Designed By : Kareem Naser Aldeen
- title: (none) -> STM32 BlueBill
